Commit message: Add laser and world

File: src/tennisbot_description/urdf/common_properties.xacro (robot description, xacro)
@@ -14,5 +14,5 @@
     </material>
     <material name="light_yellow">
-        <color rgba="0.91 0.91 0.76 1" />
+        <color rgba="0.851 0.729 0.314 1" />
     </material>
     <xacro:macro name="box_inertia" params="m x y z o_xyz o_rpy" >

File: src/tennisbot_description/urdf/tennisbot.urdf.xacro (robot description, xacro)
@@ -99,16 +99,17 @@
     <link name="IMU_link">
         <visual>
-            <origin xyz="0 0 0.01 " rpy="0 0 0"/>
+            <origin xyz="0 0 0.005 " rpy="0 0 0"/>
             <geometry>
-                <box size="0.08 0.08 0.02" />
+                <box size="0.04 0.04 0.01" />
             </geometry>
+            <material name="orange" />
         </visual>
         <collision>
-            <origin xyz="0 0 0.01 " rpy="0 0 0"/>
+            <origin xyz="0 0 0.005 " rpy="0 0 0"/>
             <geometry>
-                <box size="0.08 0.08 0.02" />
+                <box size="0.04 0.04 0.01" />
             </geometry>
         </collision>
-        <xacro:box_inertia m="0.1" x="0.08" y="0.08" z="0.02" o_xyz="0 0 0.01" o_rpy="0 0 0" />
+        <xacro:box_inertia m="0.1" x="0.04" y="0.04" z="0.01" o_xyz="0 0 0.005" o_rpy="0 0 0" />
     </link>
     <joint name="IMU_joint" type="fixed">
@@ -117,3 +118,24 @@
         <origin xyz="0.07 0 ${base_height}" rpy="0 0 0" />
     </joint>
+    <link name="laser_link">
+        <visual>
+            <geometry>
+                <cylinder radius="0.035" length="0.06" />
+            </geometry>
+            <origin xyz="0 0 0" rpy="0 0 0" />
+            <material name="blue" />
+        </visual>
+        <collision>
+            <geometry>
+                <cylinder radius="0.035" length="0.06" />
+            </geometry>
+            <origin xyz="0 0 0" rpy="0 0 0" />
+        </collision>
+        <xacro:cylinder_inertia m="0.17" r="0.035" h="0.06" o_xyz="0 0 0" o_rpy="0 0 0" />
+    </link>
+    <joint name="laser_joint" type="fixed">
+        <parent link="base_link" />
+        <child link="laser_link" />
+        <origin xyz="0 0 ${base_height}" rpy="0 0 0" />
+    </joint>
 </robot>

File: src/tennisbot_description/urdf/tennisbot_gazebo.xacro (robot description, xacro)
@@ -2,5 +2,8 @@
 <robot name="tennisbot" xmlns:xacro="http://www.ros.org/wiki/xacro">
     <gazebo reference="base_link">
-        <material>Gazebo/Yellow</material>
+        <material>
+            <ambient>0.851 0.729 0.314 1</ambient>
+            <diffuse>0.851 0.729 0.314 1</diffuse>
+        </material>
     </gazebo>
     <gazebo reference="left_wheel_link">
@@ -12,5 +15,8 @@
         <maxVel>0.1</maxVel>
         <fdir1>1 0 0</fdir1>
-        <material>Gazebo/Grey</material>
+        <material>
+            <ambient>0.5 0.5 0.5 1</ambient>
+            <diffuse>0.5 0.5 0.5 1</diffuse>
+        </material>
     </gazebo>
     <gazebo reference="right_wheel_link">
@@ -22,5 +28,8 @@
         <maxVel>0.1</maxVel>
         <fdir1>1 0 0</fdir1>
-        <material>Gazebo/Grey</material>
+        <material>
+            <ambient>0.5 0.5 0.5 1</ambient>
+            <diffuse>0.5 0.5 0.5 1</diffuse>
+        </material>
     </gazebo>
     <gazebo reference="caster_wheel_link">
@@ -31,8 +40,20 @@
         <minDepth>0.001</minDepth>
         <maxVel>0.1</maxVel>
-        <material>Gazebo/Grey</material>
+        <material>
+            <ambient>0.5 0.5 0.5 1</ambient>
+            <diffuse>0.5 0.5 0.5 1</diffuse>
+        </material>
     </gazebo>
     <gazebo reference="IMU_link">
-        <material>Gazebo/Red</material>
+        <material>
+            <ambient>1 0.5 0 1</ambient>
+            <diffuse>1 0.5 0 1</diffuse>
+        </material>
+    </gazebo>
+    <gazebo reference="laser_link">
+        <material>
+            <ambient>0 0 0.5 1</ambient>
+            <diffuse>0 0 0.5 1</diffuse>
+        </material>
     </gazebo>
     <gazebo>
@@ -43,9 +64,9 @@
         <!-- IMU -->
         <plugin filename="gz-sim-imu-system" name="gz::sim::systems::Imu"/>
+        <!-- Camera / LiDAR -->
+        <plugin filename="gz-sim-sensors-system" name="gz::sim::systems::Sensors">
+            <render_engine>ogre2</render_engine>
+        </plugin>
     </gazebo>
-        <!-- Camera / LiDAR -->
-        <!-- <plugin filename="gz-sim-sensors-system" name="gz::sim::systems::Sensors">
-            <render_engine>ogre2</render_engine>
-        </plugin> -->
      <!-- IMU -->
     <gazebo reference="IMU_link">
@@ -99,3 +120,33 @@
         </sensor>
     </gazebo>
+    <!-- 2D Laser Sensor -->
+    <gazebo reference="laser_link">
+        <sensor name="lidar" type="gpu_lidar">
+        <always_on>true</always_on>
+        <visualize>true</visualize>
+        <topic>scan</topic>
+        <update_rate>5</update_rate>
+        <gz_frame_id>laser_link</gz_frame_id>
+        <lidar>
+            <scan>
+                <horizontal>
+                    <samples>360</samples>
+                    <resolution>1.00000</resolution>
+                    <min_angle>0.000000</min_angle>
+                    <max_angle>6.280000</max_angle>
+                </horizontal>
+            </scan>
+            <range>
+                <min>0.120000</min>
+                <max>12.0</max>
+                <resolution>0.02</resolution>
+            </range>
+            <noise>
+                <type>gaussian</type>
+                <mean>0.0</mean>
+                <stddev>0.01</stddev>
+            </noise>
+        </lidar>
+        </sensor>
+    </gazebo>
 </robot>
