Commit message: urdf

File: src/tennisbot_description/urdf/tennisbot.urdf.xacro (robot description, xacro)
@@ -1,3 +1,97 @@
 <?xml version="1.0"?>
 <robot name="bumperbot" xmlns:xacro="http://www.ros.org/wiki/xacro">
+     <xacro:include filename="common_properties.xacro" />
+<!-- robot descirption -->
+    <xacro:property name="base_length" value="0.3" />
+    <xacro:property name="base_width" value="0.21" />
+    <xacro:property name="base_height" value="0.1" />
+    <xacro:property name="wheel_radius" value="0.0325" />
+    <xacro:property name="wheel_length" value="0.026" />
+    <link name="base_footprint" />
+    <link name="base_link">
+        <visual>
+            <origin xyz="0 0 ${base_height / 2.0} " rpy="0 0 0"/>
+            <geometry>
+                <box size="${base_length} ${base_width} ${base_height}" />
+            </geometry>
+            <material name="light_yellow" />
+        </visual>
+        <collision>
+            <origin xyz="0 0 ${base_height / 2.0} " rpy="0 0 0"/>
+            <geometry>
+                <box size="${base_length} ${base_width} ${base_height}" />
+            </geometry>
+        </collision>
+        <xacro:box_inertia m="2.5" x="${base_length}" y="${base_width}" z="${base_height}" o_xyz="0 0 ${base_height / 2.0}" o_rpy="0 0 0" />
+    </link>
+    <joint name="base_joint" type="fixed">
+        <parent link="base_footprint" />
+        <child link="base_link" />
+        <origin xyz="0 0 ${wheel_radius}" rpy="0 0 0" />
+    </joint>
+    <link name="left_wheel_link">
+        <visual>
+            <geometry>
+                <cylinder radius="${wheel_radius}" length="${wheel_length}" />
+            </geometry>
+            <origin xyz="0 0 0" rpy="${pi / 2.0} 0 0" />
+            <material name="grey" />
+        </visual>
+        <collision>
+            <geometry>
+                <sphere radius="${wheel_radius}" />
+            </geometry>
+            <origin xyz="0 0 0" rpy="0 0 0" />
+        </collision>
+        <xacro:cylinder_inertia m="0.5" r="${wheel_radius}" h="${wheel_length}" o_xyz="0 0 0" o_rpy="${pi / 2.0} 0 0" />
+    </link>
+    <joint name="base_leftwheel_joint" type="continuous">
+        <parent link="base_link" />
+        <child link="left_wheel_link" />
+        <origin xyz="${-(base_length / 4.0)} ${(base_width / 2.0) + (wheel_length / 2.0)} 0" rpy="0 0 0" />
+        <axis xyz="0 1 0" />
+    </joint>
+    <link name="right_wheel_link">
+        <visual>
+            <geometry>
+                <cylinder radius="${wheel_radius}" length="${wheel_length}" />
+            </geometry>
+            <origin xyz="0 0 0" rpy="${pi / 2.0} 0 0" />
+            <material name="grey" />
+        </visual>
+        <collision>
+            <geometry>
+                <sphere radius="${wheel_radius}" />
+            </geometry>
+            <origin xyz="0 0 0" rpy="0 0 0" />
+        </collision>
+        <xacro:cylinder_inertia m="0.5" r="${wheel_radius}" h="${wheel_length}" o_xyz="0 0 0" o_rpy="${pi / 2.0} 0 0" />
+    </link>
+    <joint name="base_rightwheel_joint" type="continuous">
+        <parent link="base_link" />
+        <child link="right_wheel_link" />
+        <origin xyz="${-(base_length / 4.0)} ${-(base_width / 2.0) - (wheel_length / 2.0)} 0" rpy="0 0 0" />
+        <axis xyz="0 1 0" />
+    </joint>
+    <link name="caster_wheel_link">
+        <visual>
+            <geometry>
+                <sphere radius="${wheel_radius / 2.0}" />
+            </geometry>
+            <origin xyz="0 0 0" rpy="0 0 0" />
+            <material name="grey" />
+        </visual>
+        <collision>
+            <geometry>
+                <sphere radius="${wheel_radius / 2.0}" />
+            </geometry>
+            <origin xyz="0 0 0" rpy="0 0 0" />
+        </collision>
+        <xacro:sphere_inertia m="0.25" r="${wheel_radius / 2.0}" o_xyz="0 0 0" o_rpy="0 0 0" />
+    </link>
+    <joint name="base_casterwheel_joint" type="fixed">
+        <parent link="base_link" />
+        <child link="caster_wheel_link" />
+        <origin xyz="${base_length * 3.0 / 8.0} 0 ${-wheel_radius / 2.0}" rpy="0 0 0" />
+    </joint>
 </robot>

Commit message: Add IMU

File: src/tennisbot_description/urdf/tennisbot.urdf.xacro (robot description, xacro)
@@ -97,3 +97,23 @@
         <origin xyz="${base_length * 3.0 / 8.0} 0 ${-wheel_radius / 2.0}" rpy="0 0 0" />
     </joint>
+    <link name="IMU_link">
+        <visual>
+            <origin xyz="0 0 0.01 " rpy="0 0 0"/>
+            <geometry>
+                <box size="0.08 0.08 0.02" />
+            </geometry>
+        </visual>
+        <collision>
+            <origin xyz="0 0 0.01 " rpy="0 0 0"/>
+            <geometry>
+                <box size="0.08 0.08 0.02" />
+            </geometry>
+        </collision>
+        <xacro:box_inertia m="0.1" x="0.08" y="0.08" z="0.02" o_xyz="0 0 0.01" o_rpy="0 0 0" />
+    </link>
+    <joint name="IMU_joint" type="fixed">
+        <parent link="base_link" />
+        <child link="IMU_link" />
+        <origin xyz="0.07 0 ${base_height}" rpy="0 0 0" />
+    </joint>
 </robot>

File: src/tennisbot_description/urdf/tennisbot_gazebo.xacro (robot description, xacro)
@@ -33,15 +33,69 @@
         <material>Gazebo/Grey</material>
     </gazebo>
+    <gazebo reference="IMU_link">
+        <material>Gazebo/Red</material>
+    </gazebo>
+    <gazebo>
          <!-- ROS2 Control -->
-     <gazebo>
         <plugin filename="gz_ros2_control-system" name="gz_ros2_control::GazeboSimROS2ControlPlugin">
             <parameters>$(find tennisbot_controller)/config/tennisbot_controllers.yaml</parameters>
         </plugin>
+        <!-- IMU -->
+        <plugin filename="gz-sim-imu-system" name="gz::sim::systems::Imu"/>
     </gazebo>
-        <!-- IMU -->
-        <!-- <plugin filename="gz-sim-imu-system" name="gz::sim::systems::Imu"/> -->
         <!-- Camera / LiDAR -->
         <!-- <plugin filename="gz-sim-sensors-system" name="gz::sim::systems::Sensors">
             <render_engine>ogre2</render_engine>
         </plugin> -->
+     <!-- IMU -->
+    <gazebo reference="IMU_link">
+        <sensor name="imu" type="imu">
+            <always_on>true</always_on>
+            <update_rate>100</update_rate>
+            <gz_frame_id>IMU_link</gz_frame_id>
+            <topic>imu</topic>
+            <imu>
+            <angular_velocity>
+                <x>
+                <noise type="gaussian">
+                    <mean>0.0</mean>
+                    <stddev>2e-4</stddev>
+                </noise>
+                </x>
+                <y>
+                <noise type="gaussian">
+                    <mean>0.0</mean>
+                    <stddev>2e-4</stddev>
+                </noise>
+                </y>
+                <z>
+                <noise type="gaussian">
+                    <mean>0.0</mean>
+                    <stddev>2e-4</stddev>
+                </noise>
+                </z>
+            </angular_velocity>
+            <linear_acceleration>
+                <x>
+                <noise type="gaussian">
+                    <mean>0.0</mean>
+                    <stddev>1.7e-2</stddev>
+                </noise>
+                </x>
+                <y>
+                <noise type="gaussian">
+                    <mean>0.0</mean>
+                    <stddev>1.7e-2</stddev>
+                </noise>
+                </y>
+                <z>
+                <noise type="gaussian">
+                    <mean>0.0</mean>
+                    <stddev>1.7e-2</stddev>
+                </noise>
+                </z>
+            </linear_acceleration>
+            </imu>
+        </sensor>
+    </gazebo>
 </robot>

Commit message: Add camera

File: src/tennisbot_description/urdf/tennisbot.urdf.xacro (robot description, xacro)
@@ -139,3 +139,30 @@
         <origin xyz="0 0 ${base_height}" rpy="0 0 0" />
     </joint>
+    <link name="camera_link">
+        <visual>
+            <origin xyz="0 0 0.015 " rpy="0 0 0"/>
+            <geometry>
+                <box size="0.03 0.08 0.03" />
+            </geometry>
+            <material name="orange" />
+        </visual>
+        <collision>
+            <origin xyz="0 0 0.015 " rpy="0 0 0"/>
+            <geometry>
+                <box size="0.03 0.08 0.03" />
+            </geometry>
+        </collision>
+        <xacro:box_inertia m="0.1" x="0.03" y="0.08" z="0.03" o_xyz="0 0 0.015" o_rpy="0 0 0" />
+    </link>
+    <joint name="camera_joint" type="fixed">
+        <parent link="base_link" />
+        <child link="camera_link" />
+        <origin xyz="${base_length / 2.0 + 0.015} 0 ${base_height / 2.0}" rpy="0 0 0" />
+    </joint>
+    <link name="camera_optical_link"/>
+    <joint name="camera_optical_joint" type="fixed">
+        <parent link="camera_link"/>
+        <child link="camera_optical_link"/>
+        <origin xyz="0 0 0" rpy="${-pi/2} 0 ${-pi/2}"/>
+    </joint>
 </robot>

File: src/tennisbot_description/urdf/tennisbot_gazebo.xacro (robot description, xacro)
@@ -55,4 +55,10 @@
             <ambient>0 0 0.5 1</ambient>
             <diffuse>0 0 0.5 1</diffuse>
+        </material>
+    </gazebo>
+    <gazebo reference="camera_link">
+        <material>
+            <ambient>0.1 0.1 0.1 1</ambient>
+            <diffuse>0.1 0.1 0.1 1</diffuse>
         </material>
     </gazebo>
@@ -150,3 +156,24 @@
         </sensor>
     </gazebo>
+    <!-- Camera -->
+    <gazebo reference="camera_link">
+    <sensor name="camera_sensor" type="camera">
+        <always_on>true</always_on>
+        <update_rate>30</update_rate>
+        <topic>/camera/image_raw</topic>
+        <gz_frame_id>camera_optical_link</gz_frame_id>
+        <camera>
+            <horizontal_fov>1.047</horizontal_fov>
+            <image>
+                <width>640</width>
+                <height>480</height>
+                <format>R8G8B8</format>
+            </image>
+            <clip>
+                <near>0.1</near>
+                <far>10.0</far>
+            </clip>
+        </camera>
+    </sensor>
+</gazebo>
 </robot>

Commit message: tune component size

File: src/tennisbot_description/urdf/tennisbot.urdf.xacro (robot description, xacro)
@@ -7,9 +7,10 @@
     <xacro:include filename="tennisbot_ros2_control.xacro" />
 <!-- robot descirption -->
-    <xacro:property name="base_length" value="0.3" />
-    <xacro:property name="base_width" value="0.21" />
-    <xacro:property name="base_height" value="0.1" />
-    <xacro:property name="wheel_radius" value="0.0325" />
+    <xacro:property name="base_length" value="0.25" />
+    <xacro:property name="base_width" value="0.18" />
+    <xacro:property name="base_height" value="0.068" />
+    <xacro:property name="wheel_radius" value="0.0315" />
     <xacro:property name="wheel_length" value="0.026" />
+    <xacro:property name="wheel_seperation" value="0.238" />
     <link name="base_footprint" />
     <link name="base_link">
@@ -53,5 +54,6 @@
         <parent link="base_link" />
         <child link="left_wheel_link" />
-        <origin xyz="${-(base_length / 4.0)} ${(base_width / 2.0) + (wheel_length / 2.0)} 0" rpy="0 0 0" />
+        <!-- <origin xyz="${-(base_length / 4.0)} ${(base_width / 2.0) + (wheel_length / 2.0)} 0" rpy="0 0 0" /> -->
+        <origin xyz="${-(base_length / 4.0)} ${(wheel_seperation / 2.0)} 0" rpy="0 0 0" />
         <axis xyz="0 1 0" />
     </joint>
@@ -75,5 +77,6 @@
         <parent link="base_link" />
         <child link="right_wheel_link" />
-        <origin xyz="${-(base_length / 4.0)} ${-(base_width / 2.0) - (wheel_length / 2.0)} 0" rpy="0 0 0" />
+        <!-- <origin xyz="${-(base_length / 4.0)} ${-(base_width / 2.0) - (wheel_length / 2.0)} 0" rpy="0 0 0" /> -->
+        <origin xyz="${-(base_length / 4.0)} ${-(wheel_seperation / 2.0)} 0" rpy="0 0 0" />
         <axis xyz="0 1 0" />
     </joint>

Commit message: Fix URDF

File: src/tennisbot_description/urdf/tennisbot.urdf.xacro (robot description, xacro)
@@ -81,4 +81,25 @@
         <axis xyz="0 1 0" />
     </joint>
+    <link name="support_link">
+        <visual>
+            <origin xyz="0 0 ${0.01 / 2.0} " rpy="0 0 0"/>
+            <geometry>
+                <box size="0.043 0.028 0.01" />
+            </geometry>
+            <material name="light_yellow" />
+        </visual>
+        <collision>
+            <origin xyz="0 0 ${0.003 / 2.0} " rpy="0 0 0"/>
+            <geometry>
+                <box size="0.043 0.028 0.01" />
+            </geometry>
+        </collision>
+        <xacro:box_inertia m="0.05" x="0.043" y="0.028" z="0.01" o_xyz="0 0 ${0.01 / 2.0}" o_rpy="0 0 0" />
+    </link>
+    <joint name="support_joint" type="fixed">
+        <parent link="base_link" />
+        <child link="support_link" />
+        <origin xyz="${base_length / 2.0 + 0.043 / 2.0} 0 0" rpy="0 0 0" />
+    </joint>
     <link name="caster_wheel_link">
         <visual>
@@ -100,5 +121,5 @@
         <parent link="base_link" />
         <child link="caster_wheel_link" />
-        <origin xyz="${base_length * 3.0 / 8.0} 0 ${-wheel_radius / 2.0}" rpy="0 0 0" />
+        <origin xyz="0.15 0 ${-wheel_radius / 2.0}" rpy="0 0 0" />
     </joint>
     <link name="IMU_link">

File: src/tennisbot_description/urdf/tennisbot_gazebo.xacro (robot description, xacro)
@@ -2,4 +2,10 @@
 <robot name="tennisbot" xmlns:xacro="http://www.ros.org/wiki/xacro">
     <gazebo reference="base_link">
+        <material>
+            <ambient>0.851 0.729 0.314 1</ambient>
+            <diffuse>0.851 0.729 0.314 1</diffuse>
+        </material>
+    </gazebo>
+    <gazebo reference="support_link">
         <material>
             <ambient>0.851 0.729 0.314 1</ambient>

Commit message: Adjust controller parameter

File: src/tennisbot_description/urdf/tennisbot.urdf.xacro (robot description, xacro)
@@ -90,5 +90,5 @@
         </visual>
         <collision>
-            <origin xyz="0 0 ${0.003 / 2.0} " rpy="0 0 0"/>
+            <origin xyz="0 0 ${0.01 / 2.0} " rpy="0 0 0"/>
             <geometry>
                 <box size="0.043 0.028 0.01" />

Commit message: change footprint origin

File: src/tennisbot_description/urdf/tennisbot.urdf.xacro (robot description, xacro)
@@ -33,5 +33,5 @@
         <parent link="base_footprint" />
         <child link="base_link" />
-        <origin xyz="0 0 ${wheel_radius}" rpy="0 0 0" />
+        <origin xyz="0.0625 0 ${wheel_radius}" rpy="0 0 0" />
     </joint>
     <link name="left_wheel_link">
